File: ADCS_V1/ADCS_v1.kicad_sch (KiCad schematic)
At the start: 96 parts, among them IC1 Raspberry_Pi_Zero_W__v1.3_, J1 M50-3900842, J2 M50-3902042, U1 PCA9548AD_118, U10 STSPIN250, U2 LIS3MDLTR, U3 LIS3MDLTR, U4 LIS3MDLTR, U5 LIS331DLHTR, U6 LIS331DLHTR, U7 LIS331DLHTR, U8 STSPIN250, U9 STSPIN250

Commit message: 40 pin and 16 pin def update
Connections:
- net 3.3V: now also J2.35, J2.36; no longer J2.32, J2.34
- net 5V: now also J2.39; no longer J2.38
- net GND: now also J1.3, J1.4, J2.16, J2.29, J2.3, J2.31, J2.34, J2.37, J2.38, J2.5, J2.6; no longer J1.15, J1.2, J1.7, J2.10, J2.2, J2.20, J2.25, J2.27, J2.30, J2.35, J2.36, J2.4
- net MAG_X+: now also J1.6; no longer J1.3
- net MAG_X-: now also J1.5; no longer J1.11
- net MAG_Y+: now also J1.8; no longer J1.4
- net MAG_Y-: now also J1.7; no longer J1.12
- net MAG_Z+: now also J1.10; no longer J1.13, J1.5, U10.5 (OUTA2), U10.8 (OUTB2)
- net SPIO_CS: now also J2.14; no longer J2.12
- net SPIO_MISO: now also J2.12; no longer J2.14
- net SPIO_MOSI: now also J2.10; no longer J2.16
- net SPIO_SCK: now also J2.8; no longer J2.18
- net UART1_RX: now also J2.2; no longer J2.8
- net UART1_TX: now also J2.4; no longer J2.6
- net VBAT: now also J1.13, J1.14; no longer J1.10, J1.6
- net MAG_Z-: now reaches J1.9
- net MAG_Z-: now also U10.5 (OUTA2), U10.8 (OUTB2)
- net GPIO11: no longer names the net of J2.7
- net GPIO11: no longer IC1.26 (GPIO_7/SPI0_CE2_N)
- new net GPIO1: IC1.26 (GPIO_7/SPI0_CE2_N), J2.18
- no-connect marks 55 -> 56
Other:
- moved on the sheet: J1

Commit message: changed connector positions
Parts:
- added R46: 0, Resistor_SMD:R_0402_1005Metric, symbol Device:R
- renumbered C7 to C10, C10 to C11, C3 to C12, C6 to C13, C9 to C14, C5 to C15, C8 to C16, C11 to C17, C25 to C19, C32 to C20, C19 to C21, C26 to C22, C33 to C23, C20 to C24, C27 to C25, C34 to C26, C21 to C27, C35 to C29, C12 to C3, C22 to C30, C29 to C31, C36 to C32, C23 to C33, C30 to C34, C37 to C35, C24 to C36, C31 to C37, C14 to C4, C16 to C5, C13 to C6, C15 to C7, C17 to C8, C4 to C9, J2 to J1, J1 to J2, R26 to R17, R36 to R18, R17 to R19, R27 to R20, R37 to R21, R18 to R22, R28 to R23, R38 to R24, R19 to R25, R20 to R26, R21 to R27, R29 to R28, R30 to R29, R39 to R30, R40 to R31, R31 to R32, R41 to R33, R22 to R34, R32 to R35, R42 to R36, R23 to R37, R33 to R38, R43 to R39, R24 to R40, R34 to R41, R44 to R42, R25 to R43, R45 to R44, R35 to R45
Connections:
- net 3.3V: now also J1.5, J1.6, J2.6; no longer J1.35, J1.36
- net 5V: now also J1.1, J1.2; no longer J1.39, J1.40
- net GND: now also J1.11, J1.17, J1.19, J1.26, J1.35, J1.36, J1.39, J1.4, J1.7, J1.8, J1.9, J2.13, J2.14, J2.5; no longer J1.1, J1.16, J1.21, J1.23, J1.29, J1.31, J1.33, J1.34, J1.38, J1.5, J1.6, J2.3, J2.4
- net MAG_X+: now also J2.8; no longer J2.6
- net MAG_X-: now also J2.7; no longer J2.5
- net MAG_Y+: now also J2.10; no longer J2.8
- net MAG_Y-: now also J2.9; no longer J2.7
- net MAG_Z+: now also J2.12, R46.1; no longer J2.10
- net MAG_Z-: now also J2.11, R46.2; no longer J2.9
- net SPIO_CS: now also J1.34; no longer J1.14
- net SPIO_MISO: now also J1.32; no longer J1.12
- net SPIO_MOSI: now also J1.30; no longer J1.10
- net SPIO_SCK: now also J1.28; no longer J1.8
- net UART1_RX: now also J1.38; no longer J1.2
- net UART1_TX: now also J1.40; no longer J1.4
- net VBAT: now also J2.3, J2.4; no longer J2.13, J2.14
- net GPIO1: no longer names the net of J1.18
- net GPIO1: no longer IC1.26 (GPIO_7/SPI0_CE2_N)
- new net GPIO4: IC1.26 (GPIO_7/SPI0_CE2_N), J1.16
- no-connect marks 56 -> 54
Other:
- note removed: "inductor represents magnetorquer"
